Commit message: UPDATE: changed ABB robot position

File: src/lecture_1/omtp_support/urdf/omtp_factory_assignment.xacro (robot description, xacro)
@@ -64,5 +64,5 @@
     <parent link="world_interface" />
     <child link="abbrobot_base_link" />
-    <origin xyz="0.5 -6.0 0.0" rpy="0.0 0.0 0.0"/>
+    <origin xyz="0.15 -6.0 0.0" rpy="0.0 0.0 0.0"/>
   </joint>
   <!-- gripper1 to robot1. -->

Commit message: UPDATE: Added Custom Geometry

File: src/lecture_1/omtp_support/urdf/omtp_factory_assignment.xacro (robot description, xacro)
@@ -11,5 +11,5 @@
     <origin xyz="0.5 1.8 0.0" rpy="0 0 0"/>
   </xacro:robot_pedestal_urdf>
-    <!-- Robot2 Pedestal -->
+  <!-- Robot2 Pedestal -->
   <xacro:include filename="$(find omtp_support)/urdf/robot_pedestal/robot_pedestal.urdf.xacro"/>
   <xacro:robot_pedestal_urdf pedestal_prefix="robot2_" pedestal_parent="world_interface" pedestal_height="0.95">
@@ -31,4 +31,16 @@
   <xacro:include filename="$(find omtp_support)/urdf/bin/bin.urdf.xacro"/>
   <xacro:bin_urdf prefix="bin_1_"/>
+  <!-- Custom Geometry -->
+  <link name="custom_geometry">
+    <visual>
+      <geometry>
+        <sphere radius="1"/>
+      </geometry>
+      <origin rpy="0 0 0 " xyz="0 0 1"/>
+      <material name="pink">
+        <color rgba="1 0 0.5 1"/>
+      </material>
+    </visual>
+  </link>
   <!-- Joints -->
   <joint name="world_interface_to_world" type="fixed">
@@ -44,9 +56,9 @@
   <!-- robot1 to pedestal. -->
   <joint name="robot1_to_pedestal" type="fixed">
-  <origin xyz="0 0 0.95" rpy="0 0 0" />
-  <parent link="robot1_pedestal_link" />
-  <child link="robot1_base_link" />
+    <origin xyz="0 0 0.95" rpy="0 0 0" />
+    <parent link="robot1_pedestal_link" />
+    <child link="robot1_base_link" />
   </joint>
-    <!-- robot2-pedestal to world. -->
+  <!-- robot2-pedestal to world. -->
   <joint name="robot2_pedestal_to_world_interface" type="fixed">
     <parent link="world_interface" />
@@ -56,9 +68,9 @@
   <!-- robot2 to pedestal. -->
   <joint name="robot2_to_pedestal" type="fixed">
-  <origin xyz="0 0 0.95" rpy="0 0 0" />
-  <parent link="robot2_pedestal_link" />
-  <child link="robot2_base_link" />
+    <origin xyz="0 0 0.95" rpy="0 0 0" />
+    <parent link="robot2_pedestal_link" />
+    <child link="robot2_base_link" />
   </joint>
-    <!-- abbrobot-pedestal to world. -->
+  <!-- abbrobot-pedestal to world. -->
   <joint name="abbrobot_to_world_interface" type="fixed">
     <parent link="world_interface" />
@@ -77,3 +89,9 @@
     <origin xyz="-8 -0.2 0.0" rpy="0 0 0" />
   </joint>
+  <!-- Custom Geometry -->
+  <joint name="geometry_joint" type="fixed">
+    <parent link="world_interface" />
+    <child link="custom_geometry" />
+    <origin xyz="-4 -0.2 0.0" rpy="0 0 0" />
+  </joint>
 </robot>
