Commit message: ADD: Vacuum gripper for robot two

File: lecture_1/omtp_support/urdf/omtp_factory_assignment.xacro (robot description, xacro)
@@ -28,4 +28,7 @@
   <xacro:include filename="$(find omtp_support)/urdf/vacuum_gripper/vacuum_gripper.urdf.xacro"/>
   <xacro:vacuum_gripper_urdf prefix="vacuum_gripper1_" joint_prefix="vacuum_gripper1_joint"/>
+  <!-- Vacuum Gripper2 -->
+  <xacro:include filename="$(find omtp_support)/urdf/vacuum_gripper/vacuum_gripper.urdf.xacro"/>
+  <xacro:vacuum_gripper_urdf prefix="vacuum_gripper2_" joint_prefix="vacuum_gripper2_joint"/>
   <!-- bins -->
   <xacro:include filename="$(find omtp_support)/urdf/bin/bin.urdf.xacro"/>
@@ -83,4 +86,9 @@
     <child link="vacuum_gripper1_base_link" />
   </joint>
+  <!-- gripper1 to robot1. -->
+  <joint name="gripper2_to_robot2" type="fixed">
+    <parent link="robot2_tool0" />
+    <child link="vacuum_gripper2_base_link" />
+  </joint>
   <!-- bin 1 -->
   <joint name="bin_1_joint" type="fixed">
